Commit message: Finished perceptionpipeline integration - task 4

File: catkin_ws/src/motoman/motoman_hc10_support/urdf/hc10_macro.xacro (robot description, xacro)
@@ -139,5 +139,5 @@
     </inertial>
     </link>
-    <link name="${prefix}kinect_frame">
+    <link name="kinect_frame">
     <inertial>
       <origin xyz="0 0 0" rpy="0 0 0"/>
@@ -206,8 +206,8 @@
     </joint>
     <joint type="fixed" name="effector_camera_joint">
-      <origin xyz="0.15 -1 0.1" rpy="0 0 1.57"/>
+      <origin xyz="0 0 0" rpy="1.57079632679  -1.57079632679  0"/>
       <child link="kinect_frame"/>
-      <parent link="tool0"/>
-      <axis xyz="0 0 0" rpy="0 0 0"/>
+      <parent link="${prefix}tool0"/>
+      <!--axis xyz="0 0 0" rpy="0 0 0"/-->
       <limit effort="10000" velocity="1000"/>
       <dynamics damping="1.0" friction="1.0"/>
